Commit message: Add files via upload

File: urdf/sensors.xacro (robot description, xacro)
@@ -202,5 +202,5 @@
   </xacro:macro>
 <!-- LaserScan -->
-  <xacro:macro name="laser_scanner" params="laser_name parent_link *cylinder *origin">
+  <xacro:macro name="LaserScan" params="laser_name parent_link *cylinder *origin">
     <link name="${laser_name}">
       <collision>
