Commit message: Add files via upload

File: urdf/A.urdf (robot description, URDF)
Before this commit: robot A, 11 links, 10 joints
Joints:
- joint RGB_joint: origin xyz=0 0 0.5 rpy=0 0 0 -> xyz=0 0 0.54 rpy=0 0 0
- joint arm_chassis_joint: origin xyz=0 0 0.05 rpy=0 0 0 -> xyz=0 0 0.08 rpy=0 0 0

File: urdf/robotA.urdf.xacro (robot description, xacro)
@@ -208,5 +208,5 @@
   <joint name="arm_chassis_joint" type="continuous">
       <axis xyz="0 0 1" /> <!-- Yaw -->
-      <origin rpy="0 0 0" xyz="0 0 0.05" />
+      <origin rpy="0 0 0" xyz="0 0 0.08" />
       <parent link="chassis" />
       <child link="arm_chassis" />

Commit message: Add files via upload

File: urdf/A.urdf (robot description, URDF)
Before this commit: robot A, 11 links, 10 joints
Joints:
- joint arm_chassis_joint: type fixed -> continuous

File: urdf/robotA.urdf.xacro (robot description, xacro)
@@ -196,5 +196,15 @@
     </visual>
   </link>
-  <joint name="arm_chassis_joint" type="fixed">
+  <transmission name="arm_chassis_trans">
+      <type>transmission_interface/SimpleTransmission</type>
+      <joint name="arm_chassis_joint">
+          <hardwareInterface>hardware_interface/EffortJointInterface</hardwareInterface>
+      </joint>
+      <actuator name="arm_chassis_motor">
+          <hardwareInterface>hardware_interface/EffortJointInterface</hardwareInterface>
+          <mechanicalInterface>1</mechanicalInterface>
+      </actuator>
+  </transmission>
+  <joint name="arm_chassis_joint" type="continuous">
       <axis xyz="0 0 1" />
       <origin rpy="0 0 0" xyz="0 0 0.08" />
@@ -207,5 +217,4 @@
 <!-- Arm 1 -->
   <xacro:arm number="1" posz="${arm_height/2}"/>
-  <!-- posz = 0 0 0 ???? -->
   <joint name="arm_1_joint" type="revolute">
   	<axis xyz="0 1 0"/>
