Commit message: Add files via upload

File: moveit/config/robotA.urdf.xacro (robot description, xacro)
@@ -151,5 +151,5 @@
         <origin xyz="0 0 ${posz}" rpy="0 0 0" />
         <geometry>
-          <cylinder radius="${arm_radius}" length="0.2"/>
+          <cylinder radius="${arm_radius}" length="${arm_height}"/>
         </geometry>
       </collision>
@@ -196,7 +196,15 @@
     </visual>
   </link>
+  <transmission name="arm_chassis_trans">
+      <type>transmission_interface/SimpleTransmission</type>
+      <joint name="arm_chassis_joint">
+          <hardwareInterface>hardware_interface/EffortJointInterface</hardwareInterface>
+      </joint>
+      <actuator name="arm_chassis_motor">
+          <hardwareInterface>hardware_interface/EffortJointInterface</hardwareInterface>
+          <mechanicalInterface>1</mechanicalInterface>
+      </actuator>
+  </transmission>
   <joint name="arm_chassis_joint" type="fixed">
-      <axis xyz="0 0 1" />
-      <origin rpy="0 0 0" xyz="0 0 0.08" />
       <parent link="chassis" />
       <child link="arm_chassis" />
@@ -233,12 +241,12 @@
   <xacro:include filename="$(find assignment2)/urdf/sensors.xacro"/>
 <!-- LaserScan -->
-  <xacro:LaserScan laser_name="LaserScan" parent_link="chassis">
+  <xacro:laser_scanner laser_name="LaserScan" parent_link="chassis">
     <cylinder length="0.04" radius="0.04"/>
     <origin xyz="${(chassis_length/2)} 0 ${(chassis_height/2)*1.5}" rpy="0 0 0"/>
-  </xacro:LaserScan>
+  </xacro:laser_scanner>
 <!-- RGB Camera -->
 <xacro:RGB_camera camera_name="RGB" parent_link="arm_2">
   <box size="0.08 0.08 0.08"/>
-  <origin xyz="0 0 0.34" rpy="0 0 0"/>
+  <origin xyz="0 0 ${arm_height+0.04}" rpy="0 0 0"/>
 </xacro:RGB_camera>
 <!-- GAZEBO Plugins -->
@@ -258,7 +266,7 @@
       <torque>20</torque>
       <!-- Topic to receive geometry_msgs/Twist message commands, defaults to `cmd_vel` -->
-      <commandTopic>/cmd_vel</commandTopic>
+      <commandTopic>mobile_base_controller/cmd_vel</commandTopic>
       <!-- Topic to publish nav_msgs/Odometry messages, defaults to `odom` -->
-      <odometryTopic>/odom</odometryTopic>
+      <odometryTopic>mobile_base_controller/odom</odometryTopic>
       <!-- Odometry frame, defaults to `odom` -->
       <odometryFrame>odom</odometryFrame>

File: urdf/A.urdf (robot description, URDF)
Before this commit: robot A, 11 links, 10 joints
Links:
- link arm_1: geometry collision cylinder length=0.2 radius=0.04; visual cylinder length=0.3 radius=0.04
- link arm_2: geometry collision cylinder length=0.2 radius=0.04; visual cylinder length=0.3 radius=0.04
Joints:
- joint RGB_joint: origin xyz=0 0 0.54 rpy=0 0 0 -> xyz=0 0 0.34 rpy=0 0 0
- joint arm_2_joint: origin xyz=0 0 0.5 rpy=0 0 0 -> xyz=0 0 0.3 rpy=0 0 0
- joint arm_chassis_joint: type continuous -> fixed

File: urdf/sensors.xacro (robot description, xacro)
@@ -24,5 +24,5 @@
     </link>
     <joint name="${camera_name}_joint" type="continuous">
-      <axis xyz="0 0 1" /> <!-- Yaw -->
+      <axis xyz="0 0 1" />
       <xacro:insert_block name="origin"/>
       <parent link="${parent_link}"/>
@@ -258,5 +258,5 @@
         </ray>
         <plugin name="laser_scanner_controller" filename="libgazebo_ros_laser.so">
-          <topicName>${laser_name}/laser/scan</topicName>
+          <topicName>/scan</topicName>
           <frameName>${laser_name}</frameName>
         </plugin>
